Commit message: Fix gazebo camera

File: robot_model_pkg/urdf/robot.xacro (robot description, xacro)
@@ -147,5 +147,5 @@
 	<parent link="body_link"/>
 	<child  link="camera" />
-	<origin rpy="0 0 1.57" xyz="0 0 0.08"/>
+	<origin rpy="0 0 0" xyz="0 0 0.08"/>
 </joint>
 <link name="camera">
@@ -159,5 +159,5 @@
 		<origin rpy="0 0 0" xyz="0 0 1"/>
 		<geometry>
-			<box size="0.1 0.02 0.02" />
+			<box size="0.02 0.1 0.02" />
 		</geometry>
 	</collision>

Commit message: add lidar

File: robot_model_pkg/urdf/robot.xacro (robot description, xacro)
@@ -147,9 +147,9 @@
 	<parent link="body_link"/>
 	<child  link="camera" />
-	<origin rpy="0 0 0" xyz="0 0 0.08"/>
+	<origin rpy="0 0 0" xyz="0 0 0.1"/>
 </joint>
 <link name="camera">
 	<visual>
-		<origin rpy="0 0 0" xyz="0 0 0.08"/>
+		<origin rpy="0 0 0" xyz="0 0 0.14"/>
 		<geometry>
 			<box size="0.02 0.1 0.02" />
@@ -163,3 +163,16 @@
 	</collision>
 </link>
+<joint name="hokuyo_joint" type="fixed">
+	<origin rpy="0 0 0" xyz="0 0 0.19"/>
+	<parent link="body_link"/>
+	<child link="hokuyo_link"/>
+</joint>
+<link name="hokuyo_link">
+	<visual>
+		<origin rpy="0 0 0" xyz="0 0 0"/>
+		<geometry>
+			<box size="0.2 0.2 0.08"/>
+		</geometry>
+ 	</visual>
+</link>
 </robot>

Commit message: Test version

File: robot_model_pkg/urdf/robot.xacro (robot description, xacro)
@@ -52,4 +52,23 @@
 	</inertial>
 </link>
+<joint name="before" type="fixed" >
+	<parent link="body_link"/>
+	<child  link="before_link" />
+	<origin rpy="0 0 0" xyz="0 0 0"/>
+</joint>
+<link name="before_link">
+	<visual>
+		<origin rpy="0 0 0" xyz="0.51 0 0"/>
+		<geometry>
+			<box size="0.02 0.6 0.02" />
+		</geometry>
+	</visual>
+	<collision>
+		<origin rpy="0 0 0" xyz="0 0 1"/>
+		<geometry>
+			<box size="0.02 0.6 0.02" />
+		</geometry>
+	</collision>
+</link>
 <joint name="wheel1_joint" type="continuous" >
 	<parent link="body_link"/>
@@ -134,4 +153,5 @@
 		<geometry>
 			<cylinder length="${wheel_link_length}" radius="${wheel_link_radius}"/>
+			<!-- <mesh filename="package://robot_descritpion/meshes/wheel.STL"/> -->
 		</geometry>
 	</visual>
@@ -147,9 +167,9 @@
 	<parent link="body_link"/>
 	<child  link="camera" />
-	<origin rpy="0 0 0" xyz="0 0 0.1"/>
+	<origin rpy="0 0 0" xyz="0.49 0 0.16"/>
 </joint>
 <link name="camera">
 	<visual>
-		<origin rpy="0 0 0" xyz="0 0 0.14"/>
+		<origin rpy="0 0 0" xyz="0 0 0"/>
 		<geometry>
 			<box size="0.02 0.1 0.02" />
@@ -157,5 +177,5 @@
 	</visual>
 	<collision>
-		<origin rpy="0 0 0" xyz="0 0 1"/>
+		<origin rpy="0 0 0" xyz="0 0 0"/>
 		<geometry>
 			<box size="0.02 0.1 0.02" />
@@ -176,3 +196,16 @@
  	</visual>
 </link>
+<joint name="wheel_test_j" type="fixed" >
+	<parent link="body_link"/>
+	<child  link="wheel_test_l" />
+	<origin xyz="0 0 1" rpy="0 0 0" />
+</joint>
+<link name="wheel_test_l">
+	<visual>
+		<origin rpy="1.570795 0 0" xyz="0 0 0"/>
+		<geometry>
+			<mesh filename="package://robot_model_pkg/meshes/wheel.STL"/>
+		</geometry>
+	</visual>
+</link>
 </robot>

Commit message: fix test1

File: robot_model_pkg/urdf/robot.xacro (robot description, xacro)
@@ -196,16 +196,3 @@
  	</visual>
 </link>
-<joint name="wheel_test_j" type="fixed" >
-	<parent link="body_link"/>
-	<child  link="wheel_test_l" />
-	<origin xyz="0 0 1" rpy="0 0 0" />
-</joint>
-<link name="wheel_test_l">
-	<visual>
-		<origin rpy="1.570795 0 0" xyz="0 0 0"/>
-		<geometry>
-			<mesh filename="package://robot_model_pkg/meshes/wheel.STL"/>
-		</geometry>
-	</visual>
-</link>
 </robot>

Commit message: Add map

File: robot_model_pkg/urdf/robot.xacro (robot description, xacro)
@@ -196,3 +196,16 @@
  	</visual>
 </link>
+<joint name="wheel_test_j" type="fixed" >
+	<parent link="body_link"/>
+	<child  link="wheel_test_l" />
+	<origin xyz="0 0 1" rpy="0 0 0" />
+</joint>
+<link name="wheel_test_l">
+	<visual>
+		<origin rpy="1.570795 0 0" xyz="0 0 0"/>
+		<geometry>
+			<mesh filename="package://robot_model_pkg/meshes/wheel.stl"/>
+		</geometry>
+	</visual>
+</link>
 </robot>
